File: transmitter_board/transmitter/atsamd21.kicad_sch (KiCad schematic)
At the start: 13 parts

Commit message: finished board schematic
Parts:
- gave numbers to parts that had none: 13
Connections:
- net GPIO1: now reaches U1.10 (PA05)
- net GPIO2: now reaches U1.11 (PA06)
- net GPIO3: now reaches U1.12 (PA07)
- net GPIO4: now reaches U1.13 (PA08)
- net TX: now reaches U1.15 (PA10)
- net RX: now reaches U1.16 (PA11)
- net CS1: now reaches U1.7 (PB08)
- net CS: now reaches U1.8 (PB09)
- net CS2: now reaches U1.9 (PA04)
- no-connect marks 7 -> 11
