File: transmitter_board/transmitter/bmp388.kicad_sch (KiCad schematic)
At the start: 3 parts

Commit message: finished board schematic
Parts:
- gave numbers to parts that had none: 3
Changed lines of the file:
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@@
   (symbol (lib_id "power:GND") (at 172.72 118.11 0) (unit 1)
     (in_bom yes) (on_board yes) (fields_autoplaced)
-    (property "Reference" "#PWR?" (id 0) (at 172.72 124.46 0)
+    (property "Reference" "#PWR0141" (id 0) (at 172.72 124.46 0)
       (effects (font (size 1.27 1.27)) hide)
     )
@@
   (symbol (lib_id "power:+3.3V") (at 175.26 92.71 0) (unit 1)
     (in_bom yes) (on_board yes) (fields_autoplaced)
-    (property "Reference" "#PWR?" (id 0) (at 175.26 96.52 0)
+    (property "Reference" "#PWR0138" (id 0) (at 175.26 96.52 0)
       (effects (font (size 1.27 1.27)) hide)
     )
@@
   (symbol (lib_id "power:+3.3V") (at 146.05 92.71 0) (unit 1)
     (in_bom yes) (on_board yes) (fields_autoplaced)
-    (property "Reference" "#PWR?" (id 0) (at 146.05 96.52 0)
+    (property "Reference" "#PWR0140" (id 0) (at 146.05 96.52 0)
       (effects (font (size 1.27 1.27)) hide)
     )
@@
   (symbol (lib_id "Device:C") (at 116.84 104.14 0) (unit 1)
     (in_bom yes) (on_board yes) (fields_autoplaced)
-    (property "Reference" "C?" (id 0) (at 120.65 102.8699 0)
+    (property "Reference" "C17" (id 0) (at 120.65 102.8699 0)
       (effects (font (size 1.27 1.27)) (justify left))
     )
@@
   (symbol (lib_id "power:GND") (at 146.05 118.11 0) (unit 1)
     (in_bom yes) (on_board yes) (fields_autoplaced)
-    (property "Reference" "#PWR?" (id 0) (at 146.05 124.46 0)
+    (property "Reference" "#PWR0139" (id 0) (at 146.05 124.46 0)
       (effects (font (size 1.27 1.27)) hide)
     )
@@
   (symbol (lib_id "TBC_Sensors:BMP388") (at 160.02 104.14 0) (unit 1)
     (in_bom yes) (on_board yes) (fields_autoplaced)
-    (property "Reference" "U?" (id 0) (at 160.02 91.44 0))
+    (property "Reference" "U4" (id 0) (at 160.02 91.44 0))
     (property "Value" "BMP388" (id 1) (at 160.02 93.98 0))
     (property "Footprint" "BMP388:PQFN50P200X200X80-10N" (id 2) (at 153.67 100.33 0)
@@
   (symbol (lib_id "Device:C") (at 129.54 104.14 0) (unit 1)
     (in_bom yes) (on_board yes) (fields_autoplaced)
-    (property "Reference" "C?" (id 0) (at 133.35 102.8699 0)
+    (property "Reference" "C18" (id 0) (at 133.35 102.8699 0)
       (effects (font (size 1.27 1.27)) (justify left))
     )
