File: transmitter_board/transmitter/power.kicad_sch (KiCad schematic)
At the start: 15 parts

Commit message: finished board schematic
Parts:
- added D2: SK34A, Diode_SMD:D_SMA, symbol Diode:B120-E3
- added J9: SOLAR, symbol Connector_Generic:Conn_01x02
- C10, C11: renamed from C?; value C -> 10uF
- gave numbers to parts that had none: 13
Connections:
- net GND: now also J9.1 (Pin_1)
- net VBUS: now also D2.1 (K)
- new net: D2.2 (A), J9.2 (Pin_2)
