File: transmitter_board/transmitter/regulation.kicad_sch (KiCad schematic)
At the start: 7 parts

Commit message: finished board schematic
Parts:
- gave numbers to parts that had none: 7
Changed lines of the file:
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@@
   (symbol (lib_id "Device:C") (at 113.03 107.95 0) (unit 1)
     (in_bom yes) (on_board yes) (fields_autoplaced)
-    (property "Reference" "C?" (id 0) (at 116.84 106.6799 0)
+    (property "Reference" "C15" (id 0) (at 116.84 106.6799 0)
       (effects (font (size 1.27 1.27)) (justify left))
     )
@@
   (symbol (lib_id "power:GND") (at 68.58 62.23 0) (unit 1)
     (in_bom yes) (on_board yes) (fields_autoplaced)
-    (property "Reference" "#PWR?" (id 0) (at 68.58 68.58 0)
+    (property "Reference" "#PWR0129" (id 0) (at 68.58 68.58 0)
       (effects (font (size 1.27 1.27)) hide)
     )
@@
   (symbol (lib_id "DMP3098L-7:DMP3098L-7") (at 86.36 66.04 90) (mirror x) (unit 1)
     (in_bom yes) (on_board yes) (fields_autoplaced)
-    (property "Reference" "Q?" (id 0) (at 86.36 73.66 90))
+    (property "Reference" "Q1" (id 0) (at 86.36 73.66 90))
     (property "Value" "DMP3098L-7" (id 1) (at 86.36 76.2 90))
     (property "Footprint" "DMP3098L-7:SOT91P240X110-3N" (id 2) (at 86.36 66.04 0)
@@
   (symbol (lib_id "power:GND") (at 179.07 124.46 0) (unit 1)
     (in_bom yes) (on_board yes) (fields_autoplaced)
-    (property "Reference" "#PWR?" (id 0) (at 179.07 130.81 0)
+    (property "Reference" "#PWR0133" (id 0) (at 179.07 130.81 0)
       (effects (font (size 1.27 1.27)) hide)
     )
@@
   (symbol (lib_id "Device:D_Schottky") (at 96.52 59.69 90) (unit 1)
     (in_bom yes) (on_board yes) (fields_autoplaced)
-    (property "Reference" "D?" (id 0) (at 95.5674 57.15 90)
+    (property "Reference" "D5" (id 0) (at 95.5674 57.15 90)
       (effects (font (size 1.27 1.27)) (justify right))
     )
@@
   (symbol (lib_id "power:VBUS") (at 63.5 57.15 0) (unit 1)
     (in_bom yes) (on_board yes) (fields_autoplaced)
-    (property "Reference" "#PWR?" (id 0) (at 63.5 60.96 0)
+    (property "Reference" "#PWR0130" (id 0) (at 63.5 60.96 0)
       (effects (font (size 1.27 1.27)) hide)
     )
@@
   (symbol (lib_id "power:GND") (at 191.77 124.46 0) (unit 1)
     (in_bom yes) (on_board yes) (fields_autoplaced)
-    (property "Reference" "#PWR?" (id 0) (at 191.77 130.81 0)
+    (property "Reference" "#PWR0134" (id 0) (at 191.77 130.81 0)
       (effects (font (size 1.27 1.27)) hide)
     )
@@
   (symbol (lib_id "Device:C") (at 191.77 110.49 0) (unit 1)
     (in_bom yes) (on_board yes) (fields_autoplaced)
-    (property "Reference" "C?" (id 0) (at 195.58 109.2199 0)
+    (property "Reference" "C16" (id 0) (at 195.58 109.2199 0)
       (effects (font (size 1.27 1.27)) (justify left))
     )
@@
   (symbol (lib_id "power:+3.3V") (at 191.77 96.52 0) (unit 1)
     (in_bom yes) (on_board yes) (fields_autoplaced)
-    (property "Reference" "#PWR?" (id 0) (at 191.77 100.33 0)
+    (property "Reference" "#PWR0132" (id 0) (at 191.77 100.33 0)
       (effects (font (size 1.27 1.27)) hide)
     )
@@
   (symbol (lib_id "power:GND") (at 113.03 119.38 0) (unit 1)
     (in_bom yes) (on_board yes) (fields_autoplaced)
-    (property "Reference" "#PWR?" (id 0) (at 113.03 125.73 0)
+    (property "Reference" "#PWR0131" (id 0) (at 113.03 125.73 0)
       (effects (font (size 1.27 1.27)) hide)
     )
@@
   (symbol (lib_id "Device:R") (at 74.93 59.69 270) (unit 1)
     (in_bom yes) (on_board yes) (fields_autoplaced)
-    (property "Reference" "R?" (id 0) (at 74.93 53.34 90))
+    (property "Reference" "R16" (id 0) (at 74.93 53.34 90))
     (property "Value" "4.7K" (id 1) (at 74.93 55.88 90))
     (property "Footprint" "" (id 2) (at 74.93 57.912 90)
@@
   (symbol (lib_id "Device:R") (at 83.82 53.34 180) (unit 1)
     (in_bom yes) (on_board yes) (fields_autoplaced)
-    (property "Reference" "R?" (id 0) (at 86.36 52.0699 0)
+    (property "Reference" "R17" (id 0) (at 86.36 52.0699 0)
       (effects (font (size 1.27 1.27)) (justify right))
     )
@@
   (symbol (lib_id "LP5900SD-3.3_NOPB:LP5900SD-3.3{slash}NOPB") (at 154.94 109.22 0) (unit 1)
     (in_bom yes) (on_board yes) (fields_autoplaced)
-    (property "Reference" "U?" (id 0) (at 154.94 93.98 0))
+    (property "Reference" "U3" (id 0) (at 154.94 93.98 0))
     (property "Value" "LP5900SD-3.3/NOPB" (id 1) (at 154.94 96.52 0))
     (property "Footprint" "SON65P250X220X80-7N" (id 2) (at 154.94 109.22 0)
