File: PCBs/transmitter/LTC3411.kicad_sch (KiCad schematic)
At the start: 3 parts, among them U5 LTC4311CSC6#TRPBF

Commit message: updated schematics
Parts:
- C19: footprint (none) -> Capacitor_SMD:C_0603_1608Metric
- R23: footprint (none) -> Resistor_SMD:R_0603_1608Metric
- U5: footprint SC70-SC6 -> Transistor_Power_Module:LTC4311CSC6_TRPBF
Changed lines of the file:
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@@
       (effects (font (size 1.27 1.27)) (justify left))
     )
-    (property "Footprint" "" (id 2) (at 116.5352 96.52 0)
+    (property "Footprint" "Capacitor_SMD:C_0603_1608Metric" (id 2) (at 116.5352 96.52 0)
       (effects (font (size 1.27 1.27)) hide)
     )
@@
     (property "Reference" "R23" (id 0) (at 151.13 109.22 90))
     (property "Value" "10K" (id 1) (at 151.13 111.76 90))
-    (property "Footprint" "" (id 2) (at 151.13 117.348 90)
+    (property "Footprint" "Resistor_SMD:R_0603_1608Metric" (id 2) (at 151.13 117.348 90)
       (effects (font (size 1.27 1.27)) hide)
     )
@@
     (property "Reference" "U5" (id 0) (at 152.4 78.74 0))
     (property "Value" "LTC4311CSC6#TRPBF" (id 1) (at 152.4 81.28 0))
-    (property "Footprint" "SC70-SC6" (id 2) (at 129.54 88.9 0)
+    (property "Footprint" "Transistor_Power_Module:LTC4311CSC6_TRPBF" (id 2) (at 129.54 88.9 0)
       (effects (font (size 1.27 1.27)) (justify left bottom) hide)
     )
