File: PCBs/transmitter/_autosave-transmitter.kicad_sch (KiCad schematic)
At the start: 21 parts, among them J1 Conn_01x02, J11 LoRa, J2 GPIO, J3 Ethernet, J4 Thermistor (10K), J5 RF24, J6 SWD, J7 I2C, J8 Serial, SW1 ~{RESET}

Commit message: updated schematics
Parts:
- removed H2: MountingHole, MountingHole:MountingHole_2mm, symbol Mechanical:MountingHole
Changed lines of the file:
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@@
     (pin "1")
-  )
-  (symbol (lib_id "Mechanical:MountingHole") (at 54.61 179.07 0) (unit 1)
-    (in_bom yes) (on_board yes) (fields_autoplaced)
-    (property "Reference" "H2" (id 0) (at 57.15 177.7999 0)
-      (effects (font (size 1.27 1.27)) (justify left))
-    )
-    (property "Value" "MountingHole" (id 1) (at 57.15 180.3399 0)
-      (effects (font (size 1.27 1.27)) (justify left))
-    )
-    (property "Footprint" "MountingHole:MountingHole_2mm" (id 2) (at 54.61 179.07 0)
-      (effects (font (size 1.27 1.27)) hide)
-    )
-    (property "Datasheet" "~" (id 3) (at 54.61 179.07 0)
-      (effects (font (size 1.27 1.27)) hide)
-    )
   )
   (symbol (lib_id "power:GND") (at 231.14 114.3 0) (unit 1)
@@
       (reference "H1") (unit 1) (value "MountingHole") (footprint "MountingHole:MountingHole_2mm")
     )
-    (path "/b1815453-0bc8-4e1c-801d-d1e2e330bee9"
-      (reference "H2") (unit 1) (value "MountingHole") (footprint "MountingHole:MountingHole_2mm")
-    )
     (path "/0ed3c4fe-7bb8-443a-afa1-61952af26f5a"
