File: PCBs/transmitter/bmp388.kicad_sch (KiCad schematic)
At the start: 3 parts, among them U4 BMP388

Commit message: updated schematics
Parts:
- U4: footprint BMP388:PQFN50P200X200X80-10N -> Sensor_Pressure:bmp388
Changed lines of the file:
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@@
     (property "Reference" "U4" (id 0) (at 160.02 91.44 0))
     (property "Value" "BMP388" (id 1) (at 160.02 93.98 0))
-    (property "Footprint" "BMP388:PQFN50P200X200X80-10N" (id 2) (at 153.67 100.33 0)
+    (property "Footprint" "Sensor_Pressure:bmp388" (id 2) (at 153.67 100.33 0)
       (effects (font (size 1.27 1.27)) hide)
     )
