File: PCBs/transmitter/led.kicad_sch (KiCad schematic)
At the start: 4 parts

Commit message: updated schematics
Parts:
- R20, R21, R22: footprint (none) -> Resistor_SMD:R_0603_1608Metric
Changed lines of the file:
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@@
     (property "Reference" "R20" (id 0) (at 152.4 72.39 90))
     (property "Value" "100" (id 1) (at 152.4 74.93 90))
-    (property "Footprint" "" (id 2) (at 152.4 80.518 90)
+    (property "Footprint" "Resistor_SMD:R_0603_1608Metric" (id 2) (at 152.4 80.518 90)
       (effects (font (size 1.27 1.27)) hide)
     )
@@
     (property "Reference" "R21" (id 0) (at 152.4 81.28 90))
     (property "Value" "100" (id 1) (at 152.4 86.36 90))
-    (property "Footprint" "" (id 2) (at 152.4 85.598 90)
+    (property "Footprint" "Resistor_SMD:R_0603_1608Metric" (id 2) (at 152.4 85.598 90)
       (effects (font (size 1.27 1.27)) hide)
     )
@@
     (property "Reference" "R22" (id 0) (at 152.4 91.44 90))
     (property "Value" "100" (id 1) (at 152.4 93.98 90))
-    (property "Footprint" "" (id 2) (at 152.4 90.678 90)
+    (property "Footprint" "Resistor_SMD:R_0603_1608Metric" (id 2) (at 152.4 90.678 90)
       (effects (font (size 1.27 1.27)) hide)
     )
