File: PCBs/transmitter/power.kicad_sch (KiCad schematic)
At the start: 17 parts, among them J9 SOLAR, U2 BQ24074RGT

Commit message: updated schematics
Parts:
- C10, C11, C12, C13, C14: footprint (none) -> Capacitor_SMD:C_0603_1608Metric
- D3, D4: footprint (none) -> LED_SMD:LED_0603_1608Metric
- J9: footprint (none) -> Connector_JST:JST_EH_B2B-EH-A_1x02_P2.50mm_Vertical
- R10, R11, R12, R13, R14, R15, R9: footprint (none) -> Resistor_SMD:R_0603_1608Metric
Changed lines of the file:
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@@
     (property "Reference" "R14" (id 0) (at 198.12 66.04 90))
     (property "Value" "10K" (id 1) (at 198.12 68.58 90))
-    (property "Footprint" "" (id 2) (at 198.12 74.168 90)
+    (property "Footprint" "Resistor_SMD:R_0603_1608Metric" (id 2) (at 198.12 74.168 90)
       (effects (font (size 1.27 1.27)) hide)
     )
@@
     (property "Reference" "R11" (id 0) (at 129.54 116.84 90))
     (property "Value" "1K" (id 1) (at 129.54 119.38 90))
-    (property "Footprint" "" (id 2) (at 129.54 123.698 90)
+    (property "Footprint" "Resistor_SMD:R_0603_1608Metric" (id 2) (at 129.54 123.698 90)
       (effects (font (size 1.27 1.27)) hide)
     )
@@
     (property "Reference" "D3" (id 0) (at 211.7725 66.04 0))
     (property "Value" "LED" (id 1) (at 211.7725 68.58 0))
-    (property "Footprint" "" (id 2) (at 213.36 72.39 0)
+    (property "Footprint" "LED_SMD:LED_0603_1608Metric" (id 2) (at 213.36 72.39 0)
       (effects (font (size 1.27 1.27)) hide)
     )
@@
     (property "Reference" "J9" (id 0) (at 86.36 96.52 0))
     (property "Value" "SOLAR" (id 1) (at 86.36 93.98 0))
-    (property "Footprint" "" (id 2) (at 86.36 87.63 0)
+    (property "Footprint" "Connector_JST:JST_EH_B2B-EH-A_1x02_P2.50mm_Vertical" (id 2) (at 86.36 87.63 0)
       (effects (font (size 1.27 1.27)) hide)
     )
@@
       (effects (font (size 1.27 1.27)) (justify left))
     )
-    (property "Footprint" "" (id 2) (at 186.3852 115.57 0)
+    (property "Footprint" "Capacitor_SMD:C_0603_1608Metric" (id 2) (at 186.3852 115.57 0)
       (effects (font (size 1.27 1.27)) hide)
     )
@@
       (effects (font (size 1.27 1.27)) (justify left))
     )
-    (property "Footprint" "" (id 2) (at 197.8152 115.57 0)
+    (property "Footprint" "Capacitor_SMD:C_0603_1608Metric" (id 2) (at 197.8152 115.57 0)
       (effects (font (size 1.27 1.27)) hide)
     )
@@
     (property "Reference" "R10" (id 0) (at 129.54 104.14 90))
     (property "Value" "10K" (id 1) (at 129.54 106.68 90))
-    (property "Footprint" "" (id 2) (at 129.54 110.998 90)
+    (property "Footprint" "Resistor_SMD:R_0603_1608Metric" (id 2) (at 129.54 110.998 90)
       (effects (font (size 1.27 1.27)) hide)
     )
@@
       (effects (font (size 1.27 1.27)) (justify left))
     )
-    (property "Footprint" "" (id 2) (at 87.3252 115.57 0)
+    (property "Footprint" "Capacitor_SMD:C_0603_1608Metric" (id 2) (at 87.3252 115.57 0)
       (effects (font (size 1.27 1.27)) hide)
     )
@@
     (property "Reference" "R9" (id 0) (at 129.54 93.98 90))
     (property "Value" "10K" (id 1) (at 129.54 96.52 90))
-    (property "Footprint" "" (id 2) (at 129.54 102.108 90)
+    (property "Footprint" "Resistor_SMD:R_0603_1608Metric" (id 2) (at 129.54 102.108 90)
       (effects (font (size 1.27 1.27)) hide)
     )
@@
       (effects (font (size 1.27 1.27)) (justify left))
     )
-    (property "Footprint" "" (id 2) (at 209.2452 115.57 0)
+    (property "Footprint" "Capacitor_SMD:C_0603_1608Metric" (id 2) (at 209.2452 115.57 0)
       (effects (font (size 1.27 1.27)) hide)
     )
@@
     (property "Reference" "R12" (id 0) (at 129.54 128.27 90))
     (property "Value" "1K" (id 1) (at 129.54 130.81 90))
-    (property "Footprint" "" (id 2) (at 129.54 127.508 90)
+    (property "Footprint" "Resistor_SMD:R_0603_1608Metric" (id 2) (at 129.54 127.508 90)
       (effects (font (size 1.27 1.27)) hide)
     )
@@
     (property "Reference" "D4" (id 0) (at 211.7725 77.47 0))
     (property "Value" "LED" (id 1) (at 211.7725 80.01 0))
-    (property "Footprint" "" (id 2) (at 213.36 83.82 0)
+    (property "Footprint" "LED_SMD:LED_0603_1608Metric" (id 2) (at 213.36 83.82 0)
       (effects (font (size 1.27 1.27)) hide)
     )
@@
       (effects (font (size 1.27 1.27)) (justify left))
     )
-    (property "Footprint" "" (id 2) (at 97.4852 115.57 0)
+    (property "Footprint" "Capacitor_SMD:C_0603_1608Metric" (id 2) (at 97.4852 115.57 0)
       (effects (font (size 1.27 1.27)) hide)
     )
@@
     (property "Reference" "R15" (id 0) (at 198.12 77.47 90))
     (property "Value" "10K" (id 1) (at 198.12 80.01 90))
-    (property "Footprint" "" (id 2) (at 198.12 82.042 90)
+    (property "Footprint" "Resistor_SMD:R_0603_1608Metric" (id 2) (at 198.12 82.042 90)
       (effects (font (size 1.27 1.27)) hide)
     )
@@
       (effects (font (size 1.27 1.27)) (justify right))
     )
-    (property "Footprint" "" (id 2) (at 184.658 125.73 90)
-      (effects (font (size 1.27 1.27)) hide)
-    )
+    (property "Footprint" "Resistor_SMD:R_0603_1608Metric" (id 2) (at 184.658 125.73 90)
+      (effects (font (size 1.27 1.27)) hide)
+    )
