File: PCBs/transmitter/regulation.kicad_sch (KiCad schematic)
At the start: 7 parts, among them Q1 DMP3098L-7, U3 LP5900SD-3.3/NOPB

Commit message: updated schematics
Parts:
- C15, C16: footprint (none) -> Capacitor_SMD:C_0603_1608Metric
- D5: footprint SS12:DIOM4427X270N -> Diode_SMD:1N4148
- Q1: footprint DMP3098L-7:SOT91P240X110-3N -> Transistor_Power_Module:DMP3098L
- R16, R17: footprint (none) -> Resistor_SMD:R_0603_1608Metric
- U3: footprint SON65P250X220X80-7N -> Converter_DCDC:LP5900SD-3.3_NOPB
Changed lines of the file:
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@@
       (effects (font (size 1.27 1.27)) (justify left))
     )
-    (property "Footprint" "" (id 2) (at 113.9952 111.76 0)
+    (property "Footprint" "Capacitor_SMD:C_0603_1608Metric" (id 2) (at 113.9952 111.76 0)
       (effects (font (size 1.27 1.27)) hide)
     )
@@
     (property "Reference" "Q1" (id 0) (at 86.36 73.66 90))
     (property "Value" "DMP3098L-7" (id 1) (at 86.36 76.2 90))
-    (property "Footprint" "DMP3098L-7:SOT91P240X110-3N" (id 2) (at 86.36 66.04 0)
+    (property "Footprint" "Transistor_Power_Module:DMP3098L" (id 2) (at 86.36 66.04 0)
       (effects (font (size 1.27 1.27)) (justify left bottom) hide)
     )
@@
       (effects (font (size 1.27 1.27)) (justify right))
     )
-    (property "Footprint" "SS12:DIOM4427X270N" (id 2) (at 92.71 59.69 0)
+    (property "Footprint" "Diode_SMD:1N4148" (id 2) (at 92.71 59.69 0)
       (effects (font (size 1.27 1.27)) hide)
     )
@@
       (effects (font (size 1.27 1.27)) (justify left))
     )
-    (property "Footprint" "" (id 2) (at 192.7352 114.3 0)
+    (property "Footprint" "Capacitor_SMD:C_0603_1608Metric" (id 2) (at 192.7352 114.3 0)
       (effects (font (size 1.27 1.27)) hide)
     )
@@
     (property "Reference" "R16" (id 0) (at 74.93 53.34 90))
     (property "Value" "4.7K" (id 1) (at 74.93 55.88 90))
-    (property "Footprint" "" (id 2) (at 74.93 57.912 90)
+    (property "Footprint" "Resistor_SMD:R_0603_1608Metric" (id 2) (at 74.93 57.912 90)
       (effects (font (size 1.27 1.27)) hide)
     )
@@
       (effects (font (size 1.27 1.27)) (justify right))
     )
-    (property "Footprint" "" (id 2) (at 85.598 53.34 90)
+    (property "Footprint" "Resistor_SMD:R_0603_1608Metric" (id 2) (at 85.598 53.34 90)
       (effects (font (size 1.27 1.27)) hide)
     )
@@
     (property "Reference" "U3" (id 0) (at 154.94 93.98 0))
     (property "Value" "LP5900SD-3.3/NOPB" (id 1) (at 154.94 96.52 0))
-    (property "Footprint" "SON65P250X220X80-7N" (id 2) (at 154.94 109.22 0)
+    (property "Footprint" "Converter_DCDC:LP5900SD-3.3_NOPB" (id 2) (at 154.94 109.22 0)
       (effects (font (size 1.27 1.27)) (justify left bottom) hide)
     )
