File: PCBs/main_board/TDS.kicad_sch (KiCad schematic)
At the start: 29 parts, among them J3 PROBE, U5 LM324A, U6 CD4060BM

Commit message: updated schematic labels
Other:
- title: (none) -> OceanAI
Changed lines of the file:
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@@
 (kicad_sch (version 20211123) (generator eeschema)
   (paper "A4")
+  (title_block
+    (title "OceanAI")
+    (date "2022-07-25")
+    (rev "2")
+  )
   (junction (at 182.88 130.81) (diameter 0) (color 0 0 0 0)
   )
