File: PCBs/main_board/barometer.kicad_sch (KiCad schematic)
At the start: 3 parts, among them U3 BMP388

Commit message: updated schematic labels
Other:
- title: (none) -> OceanAI
Changed lines of the file:
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@@
 (kicad_sch (version 20211123) (generator eeschema)
   (paper "A4")
+  (title_block
+    (title "OceanAI")
+    (date "2022-07-25")
+    (rev "2")
+  )
   (junction (at 132.08 113.03) (diameter 0) (color 0 0 0 0)
   )
