File: PCBs/main_board/magnetometer.kicad_sch (KiCad schematic)
At the start: 4 parts, among them U2 LIS3MDLTR

Commit message: updated schematic labels
Other:
- title: (none) -> OceanAI
Changed lines of the file:
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@@
 (kicad_sch (version 20211123) (generator eeschema)
   (paper "A4")
+  (title_block
+    (title "OceanAI")
+    (date "2022-07-25")
+    (rev "2")
+  )
   (junction (at 168.91 82.55) (diameter 0) (color 0 0 0 0)
   )
