File: PCBs/main_board/pow.kicad_sch (KiCad schematic)
At the start: 19 parts, among them Q1 DMP3098L-7, U10 LDL1117S50R, U7 MAX1719, U8 AP2112K-3.3, U9 ADP122

Commit message: updated schematic labels
Other:
- title: (none) -> OceanAI
Changed lines of the file:
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@@
 (kicad_sch (version 20211123) (generator eeschema)
   (paper "A4")
+  (title_block
+    (title "OceanAI")
+    (date "2022-07-25")
+    (rev "2")
+  )
   (junction (at 115.57 60.96) (diameter 0) (color 0 0 0 0)
   )
